Commit message: 可以在真机上运行画圆任务（粗糙）

File: se3_control/urdf/ur3.urdf (robot description, URDF)
Before this commit: robot ur3_robot, 11 links, 10 joints
Joints:
- joint flange-tool0: origin xyz=0 0 0 rpy=1.5707963267948966 0 1.5707963267948966 -> xyz=0.126 0 0 rpy=1.5707963267948966 0 1.5707963267948966
- joint shoulder_pan_joint: origin xyz=0 0 0.1519 rpy=0 0 0 -> xyz=0 0 0.1519 rpy=0 0 3.141592653589793
